Commit message: added grasp link

File: robotiq_description/urdf/robotiq_2f_85_macro.urdf.xacro (robot description, xacro)
@@ -6,4 +6,5 @@
         parent
         *origin
+        grasp_link_offset:=0.15
         sim_ignition:=false
         sim_isaac:=false
@@ -275,4 +276,10 @@
             <mimic joint="${prefix}robotiq_85_left_knuckle_joint" />
         </joint>
+        <link name="${prefix}grasp_link" />
+        <joint name="${prefix}grasp_joint" type="fixed">
+            <parent link="${prefix}robotiq_85_base_link" />
+            <child link="${prefix}grasp_link" />
+            <origin xyz="0.0 0.0 ${grasp_link_offset}" rpy="0 0 0" />
+        </joint>
     </xacro:macro>
 </robot>
